File: schematic/spotWelder/spotWelder.sch (KiCad schematic (older format))
At the start: 9 parts

Commit message: update schematic
Parts:
- added BZ?: Buzzer, symbol Device:Buzzer
- added Q?: Generic Logic N, Package_TO_SOT_SMD:SOT-323_SC-70, symbol Transistor_FET:BSS214NW
- added R?: 100, symbol Device:R
- added R?: 10k, symbol Device:R
- added U?: SSD1306-I2C-OLED-128x64, Display:EA_DOGXL160-7, symbol Display_Graphic:EA_DOGXL160-7
- D?: value DIODE -> DIODE schottky
- U?: value ATA00A18S-L -> DC/DC converter
Connections:
- net labels added: +5V
- wire segments 50 -> 73
Changed lines of the file:
@@
 P 4750 6350
 F 0 "U?" H 4750 6817 50  0000 C CNN
-F 1 "ATA00A18S-L" H 4750 6726 50  0000 C CNN
+F 1 "DC/DC converter" H 4750 6726 50  0000 C CNN
 F 2 "Converter_DCDC:Converter_DCDC_Artesyn_ATA_SMD" H 4750 6000 50  0001 C CIN
 F 3 "https://www.artesyn.com/power/assets/ata_series_ds_01apr2015_79c25814fd.pdf" H 4750 5900 50  0001 C CNN
@@
 	1    0    0    -1
 $EndComp
-$Comp
-L power:+3.3V #PWR?
-U 1 1 6053D62C
-P 5350 6050
-F 0 "#PWR?" H 5350 5900 50  0001 C CNN
-F 1 "+3.3V" H 5365 6223 50  0000 C CNN
-F 2 "" H 5350 6050 50  0001 C CNN
-F 3 "" H 5350 6050 50  0001 C CNN
-	1    5350 6050
-	1    0    0    -1
-$EndComp
-Wire Wire Line
-	5350 6050 5350 6150
 Wire Wire Line
 	5350 6150 5250 6150
@@
 P 2650 6150
 F 0 "D?" H 2650 6415 50  0000 C CNN
-F 1 "DIODE" H 2650 6324 50  0000 C CNN
+F 1 "DIODE schottky" H 2650 6324 50  0000 C CNN
 F 2 "" H 2650 6150 50  0001 C CNN
 F 3 "~" H 2650 6150 50  0001 C CNN
@@
 Wire Wire Line
 	4000 6150 4250 6150
+$Comp
+L Device:Buzzer BZ?
+U 1 1 60584C9C
+P 900 5150
+F 0 "BZ?" H 1052 5179 50  0000 L CNN
+F 1 "Buzzer" H 1052 5088 50  0000 L CNN
+F 2 "" V 875 5250 50  0001 C CNN
+F 3 "~" V 875 5250 50  0001 C CNN
+	1    900  5150
+	1    0    0    -1
+$EndComp
+$Comp
+L power:GND #PWR?
+U 1 1 60585A6D
+P 800 5850
+F 0 "#PWR?" H 800 5600 50  0001 C CNN
+F 1 "GND" H 805 5677 50  0000 C CNN
+F 2 "" H 800 5850 50  0001 C CNN
+F 3 "" H 800 5850 50  0001 C CNN
+	1    800  5850
+	1    0    0    -1
+$EndComp
+$Comp
+L Display_Graphic:EA_DOGXL160-7 U?
+U 1 1 6058DB7E
+P 4000 1500
+F 0 "U?" H 4644 1496 50  0000 L CNN
+F 1 "SSD1306-I2C-OLED-128x64" H 4644 1405 50  0000 L CNN
+F 2 "Display:EA_DOGXL160-7" H 4000 500 50  0001 C CNN
+F 3 "http://www.lcd-module.com/eng/pdf/grafik/dogxl160-7e.pdf" H 1650 2650 50  0001 C CNN
+	1    4000 1500
+	1    0    0    -1
+$EndComp
+Wire Wire Line
+	1500 3900 1800 3900
+$Comp
+L power:GND #PWR?
+U 1 1 60593E03
+P 3700 2400
+F 0 "#PWR?" H 3700 2150 50  0001 C CNN
+F 1 "GND" H 3705 2227 50  0000 C CNN
+F 2 "" H 3700 2400 50  0001 C CNN
+F 3 "" H 3700 2400 50  0001 C CNN
+	1    3700 2400
+	1    0    0    -1
+$EndComp
+Wire Wire Line
+	3700 2300 3700 2400
+$Comp
+L power:+3.3V #PWR?
+U 1 1 605967BF
+P 3200 700
+F 0 "#PWR?" H 3200 550 50  0001 C CNN
+F 1 "+3.3V" H 3215 873 50  0000 C CNN
+F 2 "" H 3200 700 50  0001 C CNN
+F 3 "" H 3200 700 50  0001 C CNN
+	1    3200 700
+	1    0    0    -1
+$EndComp
+Wire Wire Line
+	1800 4200 1150 4200
+$Comp
+L Device:R R?
+U 1 1 605B195B
+P 800 4750
+F 0 "R?" H 870 4796 50  0000 L CNN
+F 1 "100" H 870 4705 50  0000 L CNN
+F 2 "" V 730 4750 50  0001 C CNN
+F 3 "~" H 800 4750 50  0001 C CNN
+	1    800  4750
+	1    0    0    -1
+$EndComp
+$Comp
+L power:+5V #PWR?
+U 1 1 605BD90E
+P 5350 5950
+F 0 "#PWR?" H 5350 5800 50  0001 C CNN
+F 1 "+5V" H 5365 6123 50  0000 C CNN
+F 2 "" H 5350 5950 50  0001 C CNN
+F 3 "" H 5350 5950 50  0001 C CNN
+	1    5350 5950
+	1    0    0    -1
+$EndComp
+Wire Wire Line
+	5350 5950 5350 6150
+Wire Wire Line
+	3700 2300 3900 2300
+Connection ~ 3900 2300
+Wire Wire Line
+	3900 2300 4000 2300
+Wire Wire Line
+	4000 800  4000 700
+Wire Wire Line
+	4000 700  3200 700
+Wire Wire Line
+	1500 3900 1500 1200
+Wire Wire Line
+	1500 1200 3400 1200
+Wire Wire Line
+	3400 1600 1350 1600
+Wire Wire Line
+	1350 1600 1350 4000
+Wire Wire Line
+	1350 4000 1800 4000
+Wire Wire Line
+	3400 1500 1250 1500
+Wire Wire Line
+	1250 1500 1250 4100
+Wire Wire Line
+	1250 4100 1800 4100
+$Comp
+L power:+5V #PWR?
+U 1 1 605E35CF
+P 800 4500
+F 0 "#PWR?" H 800 4350 50  0001 C CNN
+F 1 "+5V" H 815 4673 50  0000 C CNN
+F 2 "" H 800 4500 50  0001 C CNN
+F 3 "" H 800 4500 50  0001 C CNN
+	1    800  4500
+	1    0    0    -1
+$EndComp
+$Comp
+L Transistor_FET:BSS214NW Q?
+U 1 1 605F3E69
+P 900 5550
+F 0 "Q?" H 1105 5596 50  0000 L CNN
+F 1 "Generic Logic N" H 250 5650 50  0000 L CNN
+F 2 "Package_TO_SOT_SMD:SOT-323_SC-70" H 1100 5475 50  0001 L CIN
+F 3 "https://www.infineon.com/dgdl/Infineon-BSS214NW-DS-v02_02-en.pdf?fileId=db3a30431b3e89eb011b695aebc01bde" H 900 5550 50  0001 L CNN
+	1    900  5550
+	-1   0    0    -1
+$EndComp
+$Comp
+L Device:R R?
+U 1 1 605F82FD
+P 1150 5700
+F 0 "R?" H 1220 5746 50  0000 L CNN
+F 1 "10k" H 1220 5655 50  0000 L CNN
+F 2 "" V 1080 5700 50  0001 C CNN
+F 3 "~" H 1150 5700 50  0001 C CNN
+	1    1150 5700
+	1    0    0    -1
+$EndComp
+Wire Wire Line
+	800  4600 800  4500
+Wire Wire Line
+	800  5050 800  4900
+Wire Wire Line
+	850  5350 800  5350
+Wire Wire Line
+	800  5350 800  5250
+Connection ~ 800  5350
+Wire Wire Line
+	1100 5550 1150 5550
+Wire Wire Line
+	1150 5850 800  5850
+Connection ~ 800  5850
+Wire Wire Line
+	1150 4200 1150 5550
+Wire Wire Line
+	800  5750 800  5850
+Connection ~ 1150 5550
 $EndSCHEMATC

Commit message: very basic menu system
Parts:
- removed Q?: Generic Logic N, Package_TO_SOT_SMD:SOT-323_SC-70, symbol Transistor_FET:BSS214NW
- added Q1: Q_NPN_BCE, symbol Device:Q_NPN_BCE
- gave numbers to parts that had none: 13
Connections:
- wire segments 73 -> 72
Changed lines of the file:
@@
 $EndDescr
 $Comp
-L MCU_ST_STM32F1:STM32F103CBTx U?
+L MCU_ST_STM32F1:STM32F103CBTx U1
 U 1 1 6052EF82
 P 2500 3600
-F 0 "U?" H 2450 2011 50  0000 C CNN
+F 0 "U1" H 2450 2011 50  0000 C CNN
 F 1 "STM32F103CBTx" H 2450 1920 50  0000 C CNN
 F 2 "Package_QFP:LQFP-48_7x7mm_P0.5mm" H 1900 2200 50  0001 R CNN
@@
 $EndComp
 $Comp
-L Device:Rotary_Encoder_Switch SW?
+L Device:Rotary_Encoder_Switch SW1
 U 1 1 60532662
 P 5300 4950
-F 0 "SW?" H 5300 5317 50  0000 C CNN
+F 0 "SW1" H 5300 5317 50  0000 C CNN
 F 1 "Rotary_Encoder_Switch" H 5300 5226 50  0000 C CNN
 F 2 "" H 5150 5110 50  0001 C CNN
@@
 $EndComp
 $Comp
-L Connector_Generic_MountingPin:Conn_01x05_MountingPin J?
+L Connector_Generic_MountingPin:Conn_01x05_MountingPin J1
 U 1 1 60533CA5
 P 2150 6350
-F 0 "J?" H 2072 6767 50  0000 C CNN
+F 0 "J1" H 2072 6767 50  0000 C CNN
 F 1 "InterBoard" H 2072 6676 50  0000 C CNN
 F 2 "" H 2150 6350 50  0001 C CNN
@@
 $EndComp
 $Comp
-L Converter_DCDC:ATA00A18S-L U?
+L Converter_DCDC:ATA00A18S-L U3
 U 1 1 60534A8D
 P 4750 6350
-F 0 "U?" H 4750 6817 50  0000 C CNN
+F 0 "U3" H 4750 6817 50  0000 C CNN
 F 1 "DC/DC converter" H 4750 6726 50  0000 C CNN
 F 2 "Converter_DCDC:Converter_DCDC_Artesyn_ATA_SMD" H 4750 6000 50  0001 C CIN
@@
 $EndComp
 $Comp
-L power:GND #PWR?
+L power:GND #PWR05
 U 1 1 6053615D
 P 2400 6800
-F 0 "#PWR?" H 2400 6550 50  0001 C CNN
+F 0 "#PWR05" H 2400 6550 50  0001 C CNN
 F 1 "GND" H 2405 6627 50  0000 C CNN
 F 2 "" H 2400 6800 50  0001 C CNN
@@
 $EndComp
 $Comp
-L power:GND #PWR?
+L power:GND #PWR010
 U 1 1 60536815
 P 4150 6650
-F 0 "#PWR?" H 4150 6400 50  0001 C CNN
+F 0 "#PWR010" H 4150 6400 50  0001 C CNN
 F 1 "GND" H 4155 6477 50  0000 C CNN
 F 2 "" H 4150 6650 50  0001 C CNN
@@
 $EndComp
 $Comp
-L power:GND #PWR?
+L power:GND #PWR03
 U 1 1 60538853
 P 2000 5100
-F 0 "#PWR?" H 2000 4850 50  0001 C CNN
+F 0 "#PWR03" H 2000 4850 50  0001 C CNN
 F 1 "GND" H 2005 4927 50  0000 C CNN
 F 2 "" H 2000 5100 50  0001 C CNN
@@
 	4150 6550 4150 6650
 $Comp
-L power:+3.3V #PWR?
+L power:+3.3V #PWR04
 U 1 1 6053BD4F
 P 2050 1850
-F 0 "#PWR?" H 2050 1700 50  0001 C CNN
+F 0 "#PWR04" H 2050 1700 50  0001 C CNN
 F 1 "+3.3V" H 2065 2023 50  0000 C CNN
 F 2 "" H 2050 1850 50  0001 C CNN
@@
 	2600 2100 2500 2100
 $Comp
-L Device:R R?
+L Device:R R3
 U 1 1 6053FC16
 P 2800 6450
-F 0 "R?" V 2950 6450 50  0000 C CNN
+F 0 "R3" V 2950 6450 50  0000 C CNN
 F 1 "470" V 2950 6600 50  0000 C CNN
 F 2 "" V 2730 6450 50  0001 C CNN
@@
 	3350 3600 3100 3600
 $Comp
-L power:GND #PWR?
+L power:GND #PWR07
 U 1 1 60555388
 P 3650 3900
-F 0 "#PWR?" H 3650 3650 50  0001 C CNN
+F 0 "#PWR07" H 3650 3650 50  0001 C CNN
 F 1 "GND" H 3655 3727 50  0000 C CNN
 F 2 "" H 3650 3900 50  0001 C CNN
@@
 $EndComp
 $Comp
-L power:GND #PWR?
+L power:GND #PWR011
 U 1 1 60556E22
 P 4850 4950
-F 0 "#PWR?" H 4850 4700 50  0001 C CNN
+F 0 "#PWR011" H 4850 4700 50  0001 C CNN
 F 1 "GND" H 4855 4777 50  0000 C CNN
 F 2 "" H 4850 4950 50  0001 C CNN
@@
 $EndComp
 $Comp
-L power:GND #PWR?
+L power:GND #PWR013
 U 1 1 6055764E
 P 5800 5050
-F 0 "#PWR?" H 5800 4800 50  0001 C CNN
+F 0 "#PWR013" H 5800 4800 50  0001 C CNN
 F 1 "GND" H 5805 4877 50  0000 C CNN
 F 2 "" H 5800 5050 50  0001 C CNN
@@
 	5850 4850 5600 4850
 $Comp
-L Device:D_Zener D?
+L Device:D_Zener D2
 U 1 1 605532B6
 P 3650 3750
-F 0 "D?" V 3604 3830 50  0000 L CNN
+F 0 "D2" V 3604 3830 50  0000 L CNN
 F 1 "3.3V" V 3695 3830 50  0000 L CNN
 F 2 "" H 3650 3750 50  0001 C CNN
@@
 GROUND
 $Comp
-L pspice:DIODE D?
+L pspice:DIODE D1
 U 1 1 6059A68B
 P 2650 6150
-F 0 "D?" H 2650 6415 50  0000 C CNN
+F 0 "D1" H 2650 6415 50  0000 C CNN
 F 1 "DIODE schottky" H 2650 6324 50  0000 C CNN
 F 2 "" H 2650 6150 50  0001 C CNN
@@
 	2850 6150 4000 6150
 $Comp
-L Device:R R?
+L Device:R R4
 U 1 1 6059FD90
 P 4150 3000
-F 0 "R?" V 4300 3000 50  0000 C CNN
+F 0 "R4" V 4300 3000 50  0000 C CNN
 F 1 "4.7k" H 4000 3000 50  0000 C CNN
 F 2 "" V 4080 3000 50  0001 C CNN
@@
 $EndComp
 $Comp
-L Device:R R?
+L Device:R R5
 U 1 1 605A0FFE
 P 4150 3400
-F 0 "R?" V 4300 3400 50  0000 C CNN
+F 0 "R5" V 4300 3400 50  0000 C CNN
 F 1 "1k" H 4000 3400 50  0000 C CNN
 F 2 "" V 4080 3400 50  0001 C CNN
@@
 $EndComp
 $Comp
-L power:GND #PWR?
+L power:GND #PWR09
 U 1 1 605A1617
 P 4150 3650
-F 0 "#PWR?" H 4150 3400 50  0001 C CNN
+F 0 "#PWR09" H 4150 3400 50  0001 C CNN
 F 1 "GND" H 4155 3477 50  0000 C CNN
 F 2 "" H 4150 3650 50  0001 C CNN
@@
 	4000 6150 4250 6150
 $Comp
-L Device:Buzzer BZ?
+L Device:Buzzer BZ1
 U 1 1 60584C9C
 P 900 5150
-F 0 "BZ?" H 1052 5179 50  0000 L CNN
+F 0 "BZ1" H 1052 5179 50  0000 L CNN
 F 1 "Buzzer" H 1052 5088 50  0000 L CNN
 F 2 "" V 875 5250 50  0001 C CNN
@@
 $EndComp
 $Comp
-L power:GND #PWR?
+L power:GND #PWR02
 U 1 1 60585A6D
 P 800 5850
-F 0 "#PWR?" H 800 5600 50  0001 C CNN
+F 0 "#PWR02" H 800 5600 50  0001 C CNN
 F 1 "GND" H 805 5677 50  0000 C CNN
 F 2 "" H 800 5850 50  0001 C CNN
@@
 $EndComp
 $Comp
-L Display_Graphic:EA_DOGXL160-7 U?
+L Display_Graphic:EA_DOGXL160-7 U2
 U 1 1 6058DB7E
 P 4000 1500
-F 0 "U?" H 4644 1496 50  0000 L CNN
+F 0 "U2" H 4644 1496 50  0000 L CNN
 F 1 "SSD1306-I2C-OLED-128x64" H 4644 1405 50  0000 L CNN
 F 2 "Display:EA_DOGXL160-7" H 4000 500 50  0001 C CNN
@@
 	1500 3900 1800 3900
 $Comp
-L power:GND #PWR?
+L power:GND #PWR08
 U 1 1 60593E03
 P 3700 2400
-F 0 "#PWR?" H 3700 2150 50  0001 C CNN
+F 0 "#PWR08" H 3700 2150 50  0001 C CNN
 F 1 "GND" H 3705 2227 50  0000 C CNN
 F 2 "" H 3700 2400 50  0001 C CNN
@@
 	3700 2300 3700 2400
 $Comp
-L power:+3.3V #PWR?
+L power:+3.3V #PWR06
 U 1 1 605967BF
 P 3200 700
-F 0 "#PWR?" H 3200 550 50  0001 C CNN
+F 0 "#PWR06" H 3200 550 50  0001 C CNN
 F 1 "+3.3V" H 3215 873 50  0000 C CNN
 F 2 "" H 3200 700 50  0001 C CNN
@@
 	1800 4200 1150 4200
 $Comp
-L Device:R R?
+L Device:R R1
 U 1 1 605B195B
 P 800 4750
-F 0 "R?" H 870 4796 50  0000 L CNN
+F 0 "R1" H 870 4796 50  0000 L CNN
 F 1 "100" H 870 4705 50  0000 L CNN
 F 2 "" V 730 4750 50  0001 C CNN
@@
 $EndComp
 $Comp
-L power:+5V #PWR?
+L power:+5V #PWR012
 U 1 1 605BD90E
 P 5350 5950
-F 0 "#PWR?" H 5350 5800 50  0001 C CNN
+F 0 "#PWR012" H 5350 5800 50  0001 C CNN
 F 1 "+5V" H 5365 6123 50  0000 C CNN
 F 2 "" H 5350 5950 50  0001 C CNN
@@
 	1250 4100 1800 4100
 $Comp
-L power:+5V #PWR?
+L power:+5V #PWR01
 U 1 1 605E35CF
 P 800 4500
-F 0 "#PWR?" H 800 4350 50  0001 C CNN
+F 0 "#PWR01" H 800 4350 50  0001 C CNN
 F 1 "+5V" H 815 4673 50  0000 C CNN
 F 2 "" H 800 4500 50  0001 C CNN
@@
 $EndComp
 $Comp
-L Transistor_FET:BSS214NW Q?
-U 1 1 605F3E69
-P 900 5550
-F 0 "Q?" H 1105 5596 50  0000 L CNN
-F 1 "Generic Logic N" H 250 5650 50  0000 L CNN
-F 2 "Package_TO_SOT_SMD:SOT-323_SC-70" H 1100 5475 50  0001 L CIN
-F 3 "https://www.infineon.com/dgdl/Infineon-BSS214NW-DS-v02_02-en.pdf?fileId=db3a30431b3e89eb011b695aebc01bde" H 900 5550 50  0001 L CNN
-	1    900  5550
-	-1   0    0    -1
-$EndComp
-$Comp
-L Device:R R?
+L Device:R R2
 U 1 1 605F82FD
 P 1150 5700
-F 0 "R?" H 1220 5746 50  0000 L CNN
+F 0 "R2" H 1220 5746 50  0000 L CNN
 F 1 "10k" H 1220 5655 50  0000 L CNN
 F 2 "" V 1080 5700 50  0001 C CNN
@@
 	800  5050 800  4900
 Wire Wire Line
-	850  5350 800  5350
-Wire Wire Line
 	800  5350 800  5250
-Connection ~ 800  5350
 Wire Wire Line
 	1100 5550 1150 5550
@@
 	800  5750 800  5850
 Connection ~ 1150 5550
+$Comp
+L Device:Q_NPN_BCE Q1
+U 1 1 60591CD0
+P 900 5550
+F 0 "Q1" H 1091 5596 50  0000 L CNN
+F 1 "Q_NPN_BCE" H 1091 5505 50  0000 L CNN
+F 2 "" H 1100 5650 50  0001 C CNN
+F 3 "~" H 900 5550 50  0001 C CNN
+	1    900  5550
+	-1   0    0    -1
+$EndComp
 $EndSCHEMATC

Commit message: add the i2c pull resistors, that fix the hang at startup
Parts:
- added R? (x2): 10k, symbol Device:R
Connections:
- net +3V3: now also R?.1, R?.1
- net at U1.42 (PB6), U2.32 (D0/SCK): now also R?.2
- net at U1.43 (PB7), U2.31 (D3/SDA): now also R?.2
Changed lines of the file:
@@
 	1500 1200 3400 1200
 Wire Wire Line
-	3400 1600 1350 1600
+	3400 1600 3100 1600
 Wire Wire Line
 	1350 1600 1350 4000
@@
 	1350 4000 1800 4000
 Wire Wire Line
-	3400 1500 1250 1500
+	3400 1500 2750 1500
 Wire Wire Line
 	1250 1500 1250 4100
@@
 	-1   0    0    -1
 $EndComp
+$Comp
+L Device:R R?
+U 1 1 605B4BC9
+P 2750 1650
+F 0 "R?" V 2900 1650 50  0000 C CNN
+F 1 "10k" H 2800 1800 50  0000 C CNN
+F 2 "" V 2680 1650 50  0001 C CNN
+F 3 "~" H 2750 1650 50  0001 C CNN
+	1    2750 1650
+	-1   0    0    1
+$EndComp
+Connection ~ 2750 1500
+Wire Wire Line
+	2750 1500 1250 1500
+$Comp
+L Device:R R?
+U 1 1 605B7597
+P 3100 1750
+F 0 "R?" V 3250 1750 50  0000 C CNN
+F 1 "10k" H 3100 1950 50  0000 C CNN
+F 2 "" V 3030 1750 50  0001 C CNN
+F 3 "~" H 3100 1750 50  0001 C CNN
+	1    3100 1750
+	-1   0    0    1
+$EndComp
+Connection ~ 3100 1600
+Wire Wire Line
+	3100 1600 1350 1600
+$Comp
+L power:+3.3V #PWR?
+U 1 1 605B7DBA
+P 2350 1900
+F 0 "#PWR?" H 2350 1750 50  0001 C CNN
+F 1 "+3.3V" H 2365 2073 50  0000 C CNN
+F 2 "" H 2350 1900 50  0001 C CNN
+F 3 "" H 2350 1900 50  0001 C CNN
+	1    2350 1900
+	1    0    0    -1
+$EndComp
+Wire Wire Line
+	2750 1800 2750 1900
+Connection ~ 2750 1900
+Wire Wire Line
+	2750 1900 3100 1900
+Wire Wire Line
+	2350 1900 2750 1900
 $EndSCHEMATC

Commit message: update kicad files
Parts:
- added Q?: SI2300 N-MOSFET, Package_TO_SOT_SMD:SOT-23, symbol Transistor_FET:ZXMN2A01F
- added R?: 10k, symbol Device:R
Connections:
- net GND: now also Q?.2 (S), R?.1
- net at U1.16 (PA6): now also Q?.1 (G), R?.2; no longer R3.1
- net at U1.18 (PB0): now also Q1.1 (B), R2.1
- new net: Q?.3 (D), R3.1
- now unconnected: U1.45 (PB8)
Changed lines of the file:
@@
 	3100 4000 3500 4000
-Wire Wire Line
-	3500 4000 3500 6450
-Wire Wire Line
-	3500 6450 2950 6450
 Wire Wire Line
 	2350 6350 3350 6350
@@
 	1    0    0    -1
 $EndComp
-Wire Wire Line
-	1800 4200 1150 4200
 $Comp
 L Device:R R1
@@
 	1150 5850 800  5850
 Connection ~ 800  5850
-Wire Wire Line
-	1150 4200 1150 5550
 Wire Wire Line
 	800  5750 800  5850
@@
 Wire Wire Line
 	2350 1900 2750 1900
+Wire Wire Line
+	1800 3400 1150 3400
+Wire Wire Line
+	1150 3400 1150 5550
+$Comp
+L Transistor_FET:ZXMN2A01F Q?
+U 1 1 605F4463
+P 3350 6750
+F 0 "Q?" H 3555 6796 50  0000 L CNN
+F 1 "SI2300 N-MOSFET" H 3555 6705 50  0000 L CNN
+F 2 "Package_TO_SOT_SMD:SOT-23" H 3550 6675 50  0001 L CIN
+F 3 "http://www.diodes.com/assets/Datasheets/ZXMN2A01F.pdf" H 3350 6750 50  0001 L CNN
+	1    3350 6750
+	-1   0    0    -1
+$EndComp
+$Comp
+L power:GND #PWR?
+U 1 1 605FAC56
+P 3250 7050
+F 0 "#PWR?" H 3250 6800 50  0001 C CNN
+F 1 "GND" H 3255 6877 50  0000 C CNN
+F 2 "" H 3250 7050 50  0001 C CNN
+F 3 "" H 3250 7050 50  0001 C CNN
+	1    3250 7050
+	1    0    0    -1
+$EndComp
+Wire Wire Line
+	3250 6550 3250 6450
+Wire Wire Line
+	3250 6450 2950 6450
+Wire Wire Line
+	3250 7050 3250 6950
+$Comp
+L Device:R R?
+U 1 1 606079F6
+P 3650 6900
+F 0 "R?" H 3550 6900 50  0000 C CNN
+F 1 "10k" H 3550 7000 50  0000 C CNN
+F 2 "" V 3580 6900 50  0001 C CNN
+F 3 "~" H 3650 6900 50  0001 C CNN
+	1    3650 6900
+	-1   0    0    1
+$EndComp
+Wire Wire Line
+	3550 6750 3650 6750
+Wire Wire Line
+	3650 7050 3250 7050
+Connection ~ 3250 7050
+Wire Wire Line
+	3500 4000 3500 6750
+Wire Wire Line
+	3500 6750 3550 6750
+Connection ~ 3550 6750
 $EndSCHEMATC
